Commit message: Update URDF and add RViz + Gazebo control configs

File: description/robot.urdf.xacro (robot description, xacro)
@@ -2,3 +2,5 @@
 <robot xmlns:xacro="http://www.ros.org/wiki/xacro" name="robot">
   <xacro:include filename="robot_core.xacro" />
+  <xacro:include filename="gazebo_control.xacro" />
+  <xacro:add_diff_drive_plugin />
 </robot>

File: description/robot_core.xacro (robot description, xacro)
@@ -41,4 +41,7 @@
     </xacro:inertial_box>
   </link>
+  <gazebo reference="chassis">
+    <material>Gazebo/White</material>
+  </gazebo>
   <!-- 3 - LINK (left wheel) -->
   <joint name="left_wheel_joint" type="continuous">
@@ -64,4 +67,7 @@
     </xacro:inertial_cylinder>
   </link>
+  <gazebo reference="left_wheel">
+    <material>Gazebo/Blue</material>
+  </gazebo>
   <!-- 3 - LINK (right wheel) -->
   <joint name="right_wheel_joint" type="continuous">
@@ -87,4 +93,7 @@
     </xacro:inertial_cylinder>
   </link>
+  <gazebo reference="right_wheel">
+    <material>Gazebo/Blue</material>
+  </gazebo>
   <!-- 4 - LINK (caster wheel) -->
   <joint name="caster_wheel_joint" type="fixed">
@@ -96,5 +105,5 @@
     <visual>
       <geometry>
-        <cylinder radius="0.05" length="0.02" />
+        <sphere radius="0.05" />
       </geometry>
       <material name="black" />
@@ -102,10 +111,15 @@
     <collision>
       <geometry>
-        <cylinder radius="0.05" length="0.02" />
+        <sphere radius="0.05" />
       </geometry>
     </collision>
-    <xacro:inertial_sphere mass="0.1" radius="0.5">
+    <xacro:inertial_sphere mass="0.1" radius="0.05">
       <origin xyz="0 0 0" rpy="0 0 0" />
     </xacro:inertial_sphere>
   </link>
+  <gazebo reference="caster_wheel">
+    <material>Gazebo/Black</material>
+    <mu1 value="0.001" />
+    <mu2 value="0.001" />
+  </gazebo>
 </robot>
