Commit message: ros2 controle plugin

File: description/depth_camera.xacro (robot description, xacro)
@@ -11,7 +11,7 @@
                 <box size="0.01 0.03 0.03" />
             </geometry>
-            <material name="red">
-                <color rgba="1 0 0 1" />
-            </material>
+            <!-- <material name="red">
+                <color rgba="1 0 0 1"/>
+            </material> -->
         </visual>
     </link>
@@ -23,6 +23,6 @@
     <link name="camera_link_optical"></link>
     <gazebo reference="camera_link">
-        <material>Gazebo/Red</material>
-        <sensor name="camera" type="camera">
+        <!-- <material>Gazebo/Red</material> -->
+        <sensor name="camera" type="depth">
             <pose>0 0 0 0 0 0</pose>
             <visualize>true</visualize>
@@ -31,5 +31,5 @@
                 <horizontal_fov>1.089</horizontal_fov>
                 <image>
-                    <format>R8G8B8</format>
+                    <format>B8G8R8</format>
                     <width>640</width>
                     <height>480</height>
@@ -42,4 +42,6 @@
             <plugin name="camera_controller" filename="libgazebo_ros_camera.so">
                 <frame_name>camera_link_optical</frame_name>
+                <min_depth>0.1</min_depth>
+                <max_depth>100.0</max_depth>
             </plugin>
         </sensor>

File: description/lidar.xacro (robot description, xacro)
@@ -12,5 +12,5 @@
                 <cylinder radius="0.05" length="0.04" />
             </geometry>
-            <material name="red" />
+            <!-- <material name="red" /> -->
         </visual>
         <collision>
@@ -48,5 +48,5 @@
                 </ros>
                 <output_type>sensor_msgs/LaserScan</output_type>
-                <frameName>laser_frame</frameName>
+                <frame_name>laser_frame</frame_name>
             </plugin>
         </sensor>

File: description/robot.urdf.xacro (robot description, xacro)
@@ -2,7 +2,8 @@
 <robot xmlns:xacro="http://www.ros.org/wiki/xacro" name="robot">
   <xacro:include filename="robot_core.xacro" />
-  <xacro:include filename="gazebo_control.xacro" />
+  <!-- <xacro:include filename="gazebo_control.xacro" /> -->
+  <xacro:include filename="ros2_control.xacro" />
   <xacro:include filename="lidar.xacro" />
   <xacro:include filename="camera.xacro" />
-  <xacro:add_diff_drive_plugin />
+  <!-- <xacro:include filename="depth_camera.xacro" /> -->
 </robot>

File: description/robot_core.xacro (robot description, xacro)
@@ -14,4 +14,7 @@
   <material name="blue">
     <color rgba="0.2 0.2 1 1" />
+  </material>
+  <material name="red">
+    <color rgba="1 0 0 1" />
   </material>
   <!-- 1 - LINK (Base) -->
