Commit message: add base_footprint link to my URDF for SLAM and NAV2

File: description/robot_core.xacro (robot description, xacro)
@@ -20,4 +20,11 @@
   <!-- 1 - LINK (Base) -->
   <link name="base_link" />
+  <!-- Base footprint link -->
+  <link name="base_footprint" />
+  <joint name="base_footprint_joint" type="fixed">
+    <parent link="base_link" />
+    <child link="base_footprint" />
+    <origin xyz="0 0 0" rpy="0 0 0" />
+  </joint>
   <!-- 2 - LINK (Chassis) -->
   <joint name="chassis_joint" type="fixed">
